Commit message: comar walking

File: resources/robots/comar/urdf/comar_a1.urdf (robot description, URDF)
Before this commit: robot comar, 18 links, 17 joints
Links:
- link comar/abad_1: geometry collision mesh filename=../meshes/ROBOT_ABDUCTION_FL.stl; visual mesh filename=../meshes/ROBOT_ABDUCTION_FL.stl
- link comar/abad_2: geometry collision mesh filename=../meshes/ROBOT_ABDUCTION_FR.stl; visual mesh filename=../meshes/ROBOT_ABDUCTION_FR.stl
- link comar/abad_3: geometry collision mesh filename=../meshes/ROBOT_ABDUCTION_HL.stl; visual mesh filename=../meshes/ROBOT_ABDUCTION_HL.stl
- link comar/abad_4: geometry collision mesh filename=../meshes/ROBOT_ABDUCTION_HR.stl; visual mesh filename=../meshes/ROBOT_ABDUCTION_HR.stl
- link comar/base_link_inertia: geometry collision box size=0.267 0.194 0.114; visual mesh filename=../meshes/ROBOT_GOVDE.stl
- link comar/hip_1: geometry collision mesh filename=../meshes/ROBOT_HIP_L.stl; visual mesh filename=../meshes/ROBOT_HIP_L.stl
- link comar/hip_2: geometry collision mesh filename=../meshes/ROBOT_HIP_R.stl; visual mesh filename=../meshes/ROBOT_HIP_R.stl
- link comar/hip_3: geometry collision mesh filename=../meshes/ROBOT_HIP_L.stl; visual mesh filename=../meshes/ROBOT_HIP_L.stl
- link comar/hip_4: geometry collision mesh filename=../meshes/ROBOT_HIP_R.stl; visual mesh filename=../meshes/ROBOT_HIP_R.stl
Joints:
- joint comar/abad_1_joint: origin xyz=222.50e-3 -65.50e-3 0 rpy=0 0 0 -> xyz=222.50e-3 65.50e-3 0 rpy=0 0 0
- joint comar/abad_2_joint: origin xyz=222.50e-3 65.50e-3 0 rpy=0 0 0 -> xyz=222.50e-3 -65.50e-3 0 rpy=0 0 0
- joint comar/abad_3_joint: origin xyz=-222.50e-3 -65.50e-3 0 rpy=0 0 0 -> xyz=-222.50e-3 65.50e-3 0 rpy=0 0 0
- joint comar/abad_4_joint: origin xyz=-222.50e-3 65.50e-3 0 rpy=0 0 0 -> xyz=-222.50e-3 -65.50e-3 0 rpy=0 0 0
- joint comar/hip_1_joint: origin xyz=0.07675 -0.0155 0  rpy=0 0 0 -> xyz=0.07675 0.0155 0  rpy=0 0 0
- joint comar/hip_2_joint: origin xyz=0.07675 0.0155 0  rpy=0 0 0 -> xyz=0.07675 -0.0155 0  rpy=0 0 0
- joint comar/hip_3_joint: origin xyz=-0.07675 -0.0155 0  rpy=0 0 0 -> xyz=-0.07675 0.0155 0  rpy=0 0 0
- joint comar/hip_4_joint: origin xyz=-0.07675 0.0155 0  rpy=0 0 0 -> xyz=-0.07675 -0.0155 0  rpy=0 0 0
- joint comar/knee_1_joint: origin xyz=0 -0.08024 -0.2  rpy=0 0 0 -> xyz=0 0.08024 -0.2  rpy=0 0 0
- joint comar/knee_2_joint: origin xyz=0 0.08024 -0.2  rpy=0 0 0 -> xyz=0 -0.08024 -0.2  rpy=0 0 0
- joint comar/knee_3_joint: origin xyz=0 -0.08024 -0.2  rpy=0 0 0 -> xyz=0 0.08024 -0.2  rpy=0 0 0
- joint comar/knee_4_joint: origin xyz=0 0.08024 -0.2  rpy=0 0 0 -> xyz=0 -0.08024 -0.2  rpy=0 0 0
